File: latex-launch-2-pcb.kicad_pcb (KiCad board)
At the start: 4 copper layers, 76.2 x 88.9 mm, 17 parts, among them J1 Conn_GPS, J2 Conn_LightAPRS-W_2.0, J3 Conn_FeatherWeight, J4 Conn_RockBLOCK, J5 Conn_GY512_MPU6050, J6 Conn_BMP280, J7 Conn_MicroSD, J8 Conn_HTU21DF

Commit message: b
Routing:
- net /I2C_SDA: track 120.1 -> 115.6 mm, vias 1 -> 0
- net /I2C_SCL: track 131.3 -> 127.8 mm
- added copper zone on In1.Cu, net GND
- added copper zone on In2.Cu, net GND
Changed lines of the file:
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@@
 	)
 	(segment
-		(start 172.212 63.734)
-		(end 172.212 70.004)
+		(start 171.704 63.226)
+		(end 171.704 69.496)
+		(width 0.4)
+		(layer "F.Cu")
+		(net 23)
+	)
+	(segment
+		(start 168.676 60.198)
+		(end 171.704 63.226)
+		(width 0.4)
+		(layer "F.Cu")
+		(net 23)
+	)
+	(segment
+		(start 171.704 69.496)
+		(end 173.312 71.104)
 		(width 0.4)
 		(layer "F.Cu")
@@
 		(start 173.312 71.104)
 		(end 175.062 71.104)
-		(width 0.4)
-		(layer "F.Cu")
-		(net 23)
-	)
-	(segment
-		(start 168.676 60.198)
-		(end 172.212 63.734)
-		(width 0.4)
-		(layer "F.Cu")
-		(net 23)
-	)
-	(segment
-		(start 172.212 70.004)
-		(end 173.312 71.104)
 		(width 0.4)
 		(layer "F.Cu")
@@
 	)
 	(segment
+		(start 173.688 67.104)
+		(end 175.062 67.104)
+		(width 0.2)
+		(layer "F.Cu")
+		(net 25)
+	)
+	(segment
 		(start 177.752 67.104)
 		(end 180.34 64.516)
@@
 		(net 25)
 	)
+	(segment
+		(start 172.974 67.818)
+		(end 173.688 67.104)
+		(width 0.2)
+		(layer "F.Cu")
+		(net 25)
+	)
 	(via
-		(at 173.482 67.056)
+		(at 172.974 67.818)
 		(size 0.6)
 		(drill 0.3)
@@
 	)
 	(segment
-		(start 180.34 64.516)
-		(end 177.8 67.056)
-		(width 0.2)
-		(layer "In2.Cu")
-		(net 25)
-	)
-	(segment
-		(start 181.61 112.395)
+		(start 172.974 67.818)
 		(end 172.974 103.759)
-		(width 0.2)
-		(layer "In2.Cu")
-		(net 25)
-	)
-	(segment
-		(start 172.974 103.759)
-		(end 172.974 71.12)
-		(width 0.2)
-		(layer "In2.Cu")
-		(net 25)
-	)
-	(segment
-		(start 177.8 67.056)
-		(end 176.53 67.056)
 		(width 0.2)
 		(layer "In2.Cu")
@@
 	)
 	(segment
-		(start 172.974 67.564)
-		(end 173.482 67.056)
+		(start 172.974 103.759)
+		(end 181.61 112.395)
 		(width 0.2)
 		(layer "In2.Cu")
@@
 	)
 	(segment
-		(start 172.974 71.12)
-		(end 172.974 67.564)
-		(width 0.2)
-		(layer "In2.Cu")
-		(net 25)
-	)
-	(segment
 		(start 178.578 69.104)
 		(end 180.34 70.866)
@@
 		(net 26)
 	)
-	(via
-		(at 176.53 69.088)
-		(size 0.6)
-		(drill 0.3)
-		(layers "F.Cu" "B.Cu")
-		(net 26)
-	)
 	(segment
 		(start 181.61 114.935)
@@
 	)
 	(segment
-		(start 180.34 70.866)
-		(end 178.562 69.088)
-		(width 0.2)
-		(layer "In2.Cu")
-		(net 26)
-	)
-	(segment
 		(start 197.136 80.486)
 		(end 214.799 62.823)
@@
 		(start 184.817 70.866)
 		(end 194.437 80.486)
-		(width 0.2)
-		(layer "In2.Cu")
-		(net 26)
-	)
-	(segment
-		(start 178.562 69.088)
-		(end 176.53 69.088)
 		(width 0.2)
 		(layer "In2.Cu")
@@
 		(net 8)
 		(net_name "GND")
-		(layer "F.Cu")
+		(layers "F.Cu" "In1.Cu" "In2.Cu")
 		(hatch edge 0.5)
 		(connect_pads

Commit message: Redid PCB; cleaner traces, design is 2 layers now
Parts:
- removed H2: MountingHole, MountingHole:MountingHole_2.7mm_M2.5_ISO7380_Pad
- C1: value C -> C10u
- moved J7 101.8 mm to (127.0, 106.7), turned to 90 degrees
- moved J1 98.1 mm to (133.1, 45.7), turned to 90 degrees
- moved J8 61.6 mm to (123.3, 82.6)
- moved R1 57.0 mm to (137.3, 91.5), turned to 90 degrees
- moved R2 53.2 mm to (137.3, 66.1), turned to -90 degrees
- moved J2 52.7 mm to (119.6, 66.9)
- moved J5 50.9 mm to (152.3, 82.1)
- moved U1 44.8 mm to (156.0, 107.9), turned to 90 degrees
- moved J4 44.4 mm to (186.2, 58.7), turned to -90 degrees
- moved R4 31.6 mm to (185.4, 44.5)
- moved R3 22.5 mm to (185.4, 52.1)
- moved H1 18.9 mm to (186.7, 35.6)
- moved J3 17.3 mm to (185.2, 95.0), turned to 90 degrees
- moved A1 16.9 mm to (180.7, 77.5), turned to 180 degrees
- moved C1 13.0 mm to (156.5, 64.8), turned to -90 degrees
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Routing:
- net +3V3: track 148.8 -> 200.0 mm, vias 1 -> 0
- net /I2C_SCL: track 127.8 -> 79.0 mm
- net /I2C_SDA: track 115.6 -> 86.2 mm, vias 0 -> 1
- net /EN_GPS: track 42.9 -> 15.2 mm
- net /SPI_SCK: track 94.0 -> 117.4 mm
- net /SPI_MISO: track 89.1 -> 112.0 mm, vias 2 -> 1
- net /Tx_iso: track 37.1 -> 59.7 mm
- net /SPI_MOSI: track 92.1 -> 109.7 mm, vias 2 -> 1
- net +BATT: track 86.9 -> 73.2 mm
- net /Rx_iso: track 38.6 -> 48.2 mm
- net /CS_RFM96W: track 64.7 -> 56.5 mm
- net /CS_SD: track 78.9 -> 71.1 mm
- net /CS_BMP280: track 59.6 -> 53.4 mm
- net Net-(A1-RX/D0): track 13.2 -> 7.02 mm
- net Net-(A1-TX/D1): track 10.4 -> 4.68 mm
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- removed copper zone on In1.Cu, net GND
- removed copper zone on In2.Cu, net GND
Other:
- outline, holes or cut-outs redrawn
- board text added: "3.5{dblquote} x 3{dblquote}"

Commit message: Added logo, added groundplane on B.Cu
Parts:
- added G***: LOGO, Latex Launch 2 Footprints:logo, F.Cu at (175.0, 89.9)
- J3: value Conn_FeatherWeight -> FeatherWeight
- moved J5 5.92 mm to (152.4, 76.2)
- moved C1 4.62 mm to (156.2, 60.2), turned to 90 degrees
Routing:
- net /I2C_SDA: track 86.2 -> 78.3 mm
- net /I2C_SCL: track 79.0 -> 83.7 mm
- net /CS_RFM96W: track 56.5 -> 58.4 mm
- net /SPI_SCK: track 117.4 -> 116.1 mm
- net /CS_SD: track 71.1 -> 69.9 mm
- net /SPI_MOSI: track 109.7 -> 108.7 mm
- net /SPI_MISO: track 112.0 -> 111.2 mm
- added copper zone on B.Cu, net GND
Other:
- outline, holes or cut-outs redrawn
- board text added: "STANFORD STUDENT SPACE INITIATIVE"

Commit message: Made changes as per design review
Parts:
- C1: value C10u -> C
- J3: value FeatherWeight -> Conn_FeatherWeight
- moved G*** 5.06 mm to (174.0, 94.9)
- moved U1 3.44 mm to (154.9, 104.6), turned to 180 degrees
- moved J6 0.88 mm to (179.7, 110.5), turned to -90 degrees
- moved J3 0.25 mm to (185.2, 94.7)
Connections:
- A1 pad 22: /CS_RFM96W -> /CS_BMP280
- A1 pad 23: /CS_BMP280 -> /CS_RFM96W
Routing:
- net /CS_BMP280: track 53.4 -> 90.3 mm, vias 0 -> 1
- net +3V3: track 199.5 -> 177.5 mm
- net /CS_RFM96W: track 58.4 -> 43.8 mm
- net /SPI_SCK: track 116.1 -> 112.8 mm
- net /SPI_MOSI: track 108.7 -> 111.3 mm
- net /I2C_SCL: track 83.7 -> 85.6 mm
- net /CS_SD: track 69.9 -> 71.6 mm
- net /SPI_MISO: track 111.2 -> 112.8 mm, vias 1 -> 0
- net /I2C_SDA: track 78.3 -> 79.8 mm

Commit message: 2nd update
Routing:
- net (no net): track 0.00 -> 21.1 mm
- net +3V3: track 177.5 -> 190.9 mm
- net /SPI_MOSI: track 111.3 -> 118.5 mm
- net /SPI_MISO: track 112.8 -> 120.0 mm
- net /SPI_SCK: track 112.8 -> 120.0 mm
- net /CS_BMP280: track 90.3 -> 87.4 mm
